Commit message: Fix inverted left-leg joint axes; add tripod gait demo to viewer
Onshape export gave left-side femur/tibia joints mirrored axes, so positive
rotation folded left legs upward — unusable with the [0, 1.75] limits. Flipped
axis signs on revolute_1_2/1_3/1_4 and revolute_2_1/2_2/2_3 so positive is the
same physical direction on all six legs. Viewer gains a walk toggle driving an
18-joint tripod gait.

Co-Authored-By: Claude Fable 5 <noreply@anthropic.com>
Claude-Session: https://claude.ai/code/session_01Srj1oQNdnN7AdjQT2ayji1

File: robot/hexapod_mkii_mock_assy/urdf/hexapod_mkii_mock_assy.urdf (robot description, URDF)
Before this commit: robot hexapod_mkii_mock_assy, 26 links, 25 joints
Joints:
- joint revolute_1_2: axis 1 -0 -0 -> -1 0 0
- joint revolute_1_3: axis 1 -0 -0 -> -1 0 0
- joint revolute_1_4: axis 1 -0 -0 -> -1 0 0
- joint revolute_2_1: axis -1 -0 -0 -> 1 0 0
- joint revolute_2_2: axis -1 -0 -0 -> 1 0 0
- joint revolute_2_3: axis -1 -0 -0 -> 1 0 0
