Commit message: Re-home the six M4 lever hub bolts to the push lever
User-verified: Onshape M4 8mm instances <1>-<6> are hard-joined to the
tibia push lever; added as a scoped override so they rotate with the
lever instead of the femur.

Co-Authored-By: Claude Opus 5 <noreply@anthropic.com>

File: robot/hexapod_leg_v3/urdf/leg_v3_linkage.urdf (robot description, URDF)
Before this commit: robot leg_v3_linkage, 6 links, 5 joints
Links:
- link femur: geometry collision box size=0.13967284 0.14347241 0.062301016; visual mesh filename=package://hexapod_leg_v3/meshes/0001755650_00mini_000_asm_1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
- link tibia_push_lever: geometry collision box size=0.031655657 0.049877248 0.017102033; visual mesh filename=package://hexapod_leg_v3/meshes/0001755650_00mini_000_asm_1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

Commit message: Re-home the six M4 hip bolts, output flange, and rotor to the coxa
User-verified: the coxa subassembly's M4 8mm <1>-<6> are rigid to the
coxa; the hip motor's output flange and rotor bolt to the coxa through
them, so all eight parts now hold still while the femur pitches. Femur
hinge added to the joint-bore audit.

Co-Authored-By: Claude Opus 5 <noreply@anthropic.com>

File: robot/hexapod_leg_v3/urdf/leg_v3_linkage.urdf (robot description, URDF)
Before this commit: robot leg_v3_linkage, 6 links, 5 joints
Links:
- link coxa: geometry collision box size=0.10611369 0.062300101 0.052756505; visual mesh filename=package://hexapod_leg_v3/meshes/0001755650_00mini_000_asm_1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
- link femur: geometry collision box size=0.13967284 0.14347241 0.05865082; visual mesh filename=package://hexapod_leg_v3/meshes/0001755652_00mini_000_asm_1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

File: robot/hexapod_leg_v3/urdf/leg_v3_serial.urdf (robot description, URDF)
Before this commit: robot leg_v3_serial, 4 links, 3 joints
Links:
- link coxa: geometry collision box size=0.10611369 0.062300101 0.052756505; visual mesh filename=package://hexapod_leg_v3/meshes/0001755650_00mini_000_asm_1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
- link femur: geometry collision box size=0.13967284 0.16207961 0.05865082; visual mesh filename=package://hexapod_leg_v3/meshes/0001755650_00mini_000_asm_1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

Commit message: Re-home the six -y knee mount screws to the femur
User-verified: Onshape M3 6mm <21>-<26> are bonded to the femur plate;
both knee bolt-circle faces now hold still through the tibia sweep.

Co-Authored-By: Claude Opus 5 <noreply@anthropic.com>

File: robot/hexapod_leg_v3/urdf/leg_v3_linkage.urdf (robot description, URDF)
Before this commit: robot leg_v3_linkage, 6 links, 5 joints
Links:
- link femur: geometry collision box size=0.13967284 0.14347241 0.05865082; visual mesh filename=package://hexapod_leg_v3/meshes/0001755652_00mini_000_asm_1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
- link tibia: geometry collision box size=0.14352877 0.25284988 0.049001406; visual mesh filename=package://hexapod_leg_v3/meshes/bearing_insert.stl

File: robot/hexapod_leg_v3/urdf/leg_v3_serial.urdf (robot description, URDF)
Before this commit: robot leg_v3_serial, 4 links, 3 joints
Links:
- link femur: geometry collision box size=0.13967284 0.16207961 0.05865082; visual mesh filename=package://hexapod_leg_v3/meshes/0001755650_00mini_000_asm_1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
- link tibia: geometry collision box size=0.14352877 0.25284988 0.049001406; visual mesh filename=package://hexapod_leg_v3/meshes/bearing_insert.stl

Commit message: Unify all six M4 4mm hip screws to the coxa
User-verified: the whole M4 4mm bolt circle is under the coxa subassy;
three were still rotating with the femur.

Co-Authored-By: Claude Opus 5 <noreply@anthropic.com>

File: robot/hexapod_leg_v3/urdf/leg_v3_linkage.urdf (robot description, URDF)
Before this commit: robot leg_v3_linkage, 6 links, 5 joints
Links:
- link coxa: geometry collision box size=0.10611369 0.062300101 0.052756505; visual mesh filename=package://hexapod_leg_v3/meshes/0001755650_00mini_000_asm_1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
- link femur: geometry collision box size=0.13967284 0.14347241 0.054100943; visual mesh filename=package://hexapod_leg_v3/meshes/0001755652_00mini_000_asm_1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

File: robot/hexapod_leg_v3/urdf/leg_v3_serial.urdf (robot description, URDF)
Before this commit: robot leg_v3_serial, 4 links, 3 joints
Links:
- link coxa: geometry collision box size=0.10611369 0.062300101 0.052756505; visual mesh filename=package://hexapod_leg_v3/meshes/0001755650_00mini_000_asm_1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
- link femur: geometry collision box size=0.13967284 0.16207961 0.056098607; visual mesh filename=package://hexapod_leg_v3/meshes/0001755650_00mini_000_asm_1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

Commit message: Remove coxa_yaw from the leg reference; manual drag control by default
The yaw DOF is the chassis<->leg interface, not internal to the leg:
leg_base merges into the coxa (single root link, 2-DOF reference) and
the yaw axis moves to leg_reference.json's body_interface record for
the six-leg assembly import. The preview defaults to manual mode with
two motor sliders (motor 3 commands the lever; knee output derived).

Co-Authored-By: Claude Opus 5 <noreply@anthropic.com>

File: robot/hexapod_leg_v3/urdf/leg_v3_linkage.urdf (robot description, URDF)
Before this commit: robot leg_v3_linkage, 6 links, 5 joints
Links:
- removed link leg_base
- link coxa: mass 0.11989778 -> 0.21655167; geometry collision box size=0.1071656 0.062300101 0.056501885; visual mesh filename=package://hexapod_leg_v3/meshes/0001755650_00mini_000_asm_1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
Joints:
- removed joint coxa_yaw
- joint femur_pitch: origin xyz=-0.048999154 0.025001668 -0.025500029 rpy=-1.5708058 6.5896378e-05 -3.4193211e-05 -> xyz=-0.048999154 -0.025001668 0.025500029 rpy=1.5707869 -6.5896378e-05 3.4193211e-05

File: robot/hexapod_leg_v3/urdf/leg_v3_serial.urdf (robot description, URDF)
Before this commit: robot leg_v3_serial, 4 links, 3 joints
Links:
- removed link leg_base
- link coxa: mass 0.11989778 -> 0.21655167; geometry collision box size=0.1071656 0.062300101 0.056501885; visual mesh filename=package://hexapod_leg_v3/meshes/0001755650_00mini_000_asm_1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
Joints:
- removed joint coxa_yaw
- joint femur_pitch: origin xyz=-0.048999154 0.025001668 -0.025500029 rpy=-1.5708058 6.5896378e-05 -3.4193211e-05 -> xyz=-0.048999154 -0.025001668 0.025500029 rpy=1.5707869 -6.5896378e-05 3.4193211e-05
