Commit message: Bond the tibia pushrod cover to the push lever
User-verified: the cover is rigidly attached to the push lever, not to the
pushrod it covers. Added as a part_overrides.json rule; URDFs and the
assembly report regenerated (lever 54.7 g, pushrod 32.9 g per leg).

Co-Authored-By: Claude Fable 5.1 <noreply@anthropic.com>

File: robot/hexapod_mkii_assy/urdf/hexapod_mkii_linkage.urdf (robot description, URDF)
Before this commit: robot hexapod_mkii_linkage, 31 links, 30 joints
Links:
- link lf_tibia_push_lever: mass 0.051266454 -> 0.054741785; geometry collision box size=0.004748708 0.030901565 0.051467069; collision box size=0.0087104031 0.031523677 0.051667737
- link lf_tibia_pushrod: mass 0.036356473 -> 0.032881142; geometry collision box size=0.010819785 0.012035149 0.089397284; visual mesh filename=package://hexapod_mkii_assy/meshes/cut_extrude2.stl
- link lm_tibia_push_lever: mass 0.051266454 -> 0.054741785; geometry collision box size=0.004748708 0.030901565 0.051467069; collision box size=0.0087104031 0.031523677 0.051667737
- link lm_tibia_pushrod: mass 0.036356473 -> 0.032881142; geometry collision box size=0.010819785 0.012035149 0.089397284; visual mesh filename=package://hexapod_mkii_assy/meshes/cut_extrude2.stl
- link lr_tibia_push_lever: mass 0.051266454 -> 0.054741785; geometry collision box size=0.004748708 0.030901565 0.051467069; collision box size=0.0087104031 0.031523677 0.051667737
- link lr_tibia_pushrod: mass 0.036356473 -> 0.032881142; geometry collision box size=0.010819785 0.012035149 0.089397284; visual mesh filename=package://hexapod_mkii_assy/meshes/cut_extrude2.stl
- link rf_tibia_push_lever: mass 0.051266454 -> 0.054741785; geometry collision box size=0.004748708 0.030901565 0.051467069; collision box size=0.0087104031 0.031523677 0.051667737
- link rf_tibia_pushrod: mass 0.036356473 -> 0.032881142; geometry collision box size=0.010819785 0.012035149 0.089397284; visual mesh filename=package://hexapod_mkii_assy/meshes/cut_extrude2.stl
- link rm_tibia_push_lever: mass 0.051266454 -> 0.054741785; geometry collision box size=0.004748708 0.030901565 0.051467069; collision box size=0.0087104031 0.031523677 0.051667737
- link rm_tibia_pushrod: mass 0.036356473 -> 0.032881142; geometry collision box size=0.010819785 0.012035149 0.089397284; visual mesh filename=package://hexapod_mkii_assy/meshes/cut_extrude2.stl
- link rr_tibia_push_lever: mass 0.051266454 -> 0.054741785; geometry collision box size=0.004748708 0.030901565 0.051467069; collision box size=0.0087104031 0.031523677 0.051667737
- link rr_tibia_pushrod: mass 0.036356473 -> 0.032881142; geometry collision box size=0.010819785 0.012035149 0.089397284; visual mesh filename=package://hexapod_mkii_assy/meshes/cut_extrude2.stl

Commit message: Point the Isaac Lab task at the CAD assembly and derive its limits and stance
The URDF's femur/tibia signs differ from the mock (positive femur raises the
leg, positive tibia opens the knee, zero is the CAD pose), so the mock's
0..1.745 / 0..2.53 ranges and 0.4 / 2.1 stance would fold the legs above the
body. Limits are now derived from the CAD kinematics (femur -1.745..0.55,
tibia -0.95..1.75, robot/hexapod_mkii_assy/joint_limits.json) and the
reset stance is femur -0.25 / tibia -0.55 with the bottom plate 0.124 m up
(stance.json), which balances static hip and knee torque at 0.9 N*m for
the 8.26 kg assembly. asset_cfg/env_cfg use the lf..rr link and joint
names, the body root, the nested Geometry/body contact-sensor paths, the
new USD path and the pad-based distal-foot threshold; the validator and
checkpoint evaluator take their angle ranges from the asset config; the
phase-3 sensor mounts follow the root link; the stance sweep carries
candidates for the new asset. tools/import_urdf_to_usd.py imports the URDF
headlessly with Isaac Sim (URDF inertials kept, primitives, floating base)
and the viewer gains the stance pose. 288 unit tests pass.

Co-Authored-By: Claude Fable 5.1 <noreply@anthropic.com>

File: robot/hexapod_mkii_assy/urdf/hexapod_mkii_linkage.urdf (robot description, URDF)
Before this commit: robot hexapod_mkii_linkage, 31 links, 30 joints
Joints:
- joint lf_femur_pitch: limit lower=0.0 upper=1.74533 effort=5.5 velocity=50.26548246 -> lower=-1.745329 upper=0.55 effort=5.5 velocity=50.26548246
- joint lf_tibia_lever_pivot: limit lower=-2.53073 upper=2.53073 effort=0.5 velocity=50.26548246 -> lower=-1.75 upper=1.75 effort=0.5 velocity=50.26548246
- joint lf_tibia_pitch: limit lower=0.0 upper=2.53073 effort=5.5 velocity=50.26548246 -> lower=-0.95 upper=1.75 effort=5.5 velocity=50.26548246
- joint lf_tibia_rod_pivot: limit lower=-2.53073 upper=2.53073 effort=0.5 velocity=50.26548246 -> lower=-1.75 upper=1.75 effort=0.5 velocity=50.26548246
- joint lm_femur_pitch: limit lower=0.0 upper=1.74533 effort=5.5 velocity=50.26548246 -> lower=-1.745329 upper=0.55 effort=5.5 velocity=50.26548246
- joint lm_tibia_lever_pivot: limit lower=-2.53073 upper=2.53073 effort=0.5 velocity=50.26548246 -> lower=-1.75 upper=1.75 effort=0.5 velocity=50.26548246
- joint lm_tibia_pitch: limit lower=0.0 upper=2.53073 effort=5.5 velocity=50.26548246 -> lower=-0.95 upper=1.75 effort=5.5 velocity=50.26548246
- joint lm_tibia_rod_pivot: limit lower=-2.53073 upper=2.53073 effort=0.5 velocity=50.26548246 -> lower=-1.75 upper=1.75 effort=0.5 velocity=50.26548246
- joint lr_femur_pitch: limit lower=0.0 upper=1.74533 effort=5.5 velocity=50.26548246 -> lower=-1.745329 upper=0.55 effort=5.5 velocity=50.26548246
- joint lr_tibia_lever_pivot: limit lower=-2.53073 upper=2.53073 effort=0.5 velocity=50.26548246 -> lower=-1.75 upper=1.75 effort=0.5 velocity=50.26548246
- joint lr_tibia_pitch: limit lower=0.0 upper=2.53073 effort=5.5 velocity=50.26548246 -> lower=-0.95 upper=1.75 effort=5.5 velocity=50.26548246
- joint lr_tibia_rod_pivot: limit lower=-2.53073 upper=2.53073 effort=0.5 velocity=50.26548246 -> lower=-1.75 upper=1.75 effort=0.5 velocity=50.26548246
- joint rf_femur_pitch: limit lower=0.0 upper=1.74533 effort=5.5 velocity=50.26548246 -> lower=-1.745329 upper=0.55 effort=5.5 velocity=50.26548246
- joint rf_tibia_lever_pivot: limit lower=-2.53073 upper=2.53073 effort=0.5 velocity=50.26548246 -> lower=-1.75 upper=1.75 effort=0.5 velocity=50.26548246
- joint rf_tibia_pitch: limit lower=0.0 upper=2.53073 effort=5.5 velocity=50.26548246 -> lower=-0.95 upper=1.75 effort=5.5 velocity=50.26548246
- joint rf_tibia_rod_pivot: limit lower=-2.53073 upper=2.53073 effort=0.5 velocity=50.26548246 -> lower=-1.75 upper=1.75 effort=0.5 velocity=50.26548246
- joint rm_femur_pitch: limit lower=0.0 upper=1.74533 effort=5.5 velocity=50.26548246 -> lower=-1.745329 upper=0.55 effort=5.5 velocity=50.26548246
- joint rm_tibia_lever_pivot: limit lower=-2.53073 upper=2.53073 effort=0.5 velocity=50.26548246 -> lower=-1.75 upper=1.75 effort=0.5 velocity=50.26548246
- joint rm_tibia_pitch: limit lower=0.0 upper=2.53073 effort=5.5 velocity=50.26548246 -> lower=-0.95 upper=1.75 effort=5.5 velocity=50.26548246
- joint rm_tibia_rod_pivot: limit lower=-2.53073 upper=2.53073 effort=0.5 velocity=50.26548246 -> lower=-1.75 upper=1.75 effort=0.5 velocity=50.26548246
- joint rr_femur_pitch: limit lower=0.0 upper=1.74533 effort=5.5 velocity=50.26548246 -> lower=-1.745329 upper=0.55 effort=5.5 velocity=50.26548246
- joint rr_tibia_lever_pivot: limit lower=-2.53073 upper=2.53073 effort=0.5 velocity=50.26548246 -> lower=-1.75 upper=1.75 effort=0.5 velocity=50.26548246
- joint rr_tibia_pitch: limit lower=0.0 upper=2.53073 effort=5.5 velocity=50.26548246 -> lower=-0.95 upper=1.75 effort=5.5 velocity=50.26548246
- joint rr_tibia_rod_pivot: limit lower=-2.53073 upper=2.53073 effort=0.5 velocity=50.26548246 -> lower=-1.75 upper=1.75 effort=0.5 velocity=50.26548246

File: robot/hexapod_mkii_assy/urdf/hexapod_mkii_serial.urdf (robot description, URDF)
Before this commit: robot hexapod_mkii_serial, 19 links, 18 joints
Joints:
- joint lf_femur_pitch: limit lower=0.0 upper=1.74533 effort=5.5 velocity=50.26548246 -> lower=-1.745329 upper=0.55 effort=5.5 velocity=50.26548246
- joint lf_tibia_pitch: limit lower=0.0 upper=2.53073 effort=5.5 velocity=50.26548246 -> lower=-0.95 upper=1.75 effort=5.5 velocity=50.26548246
- joint lm_femur_pitch: limit lower=0.0 upper=1.74533 effort=5.5 velocity=50.26548246 -> lower=-1.745329 upper=0.55 effort=5.5 velocity=50.26548246
- joint lm_tibia_pitch: limit lower=0.0 upper=2.53073 effort=5.5 velocity=50.26548246 -> lower=-0.95 upper=1.75 effort=5.5 velocity=50.26548246
- joint lr_femur_pitch: limit lower=0.0 upper=1.74533 effort=5.5 velocity=50.26548246 -> lower=-1.745329 upper=0.55 effort=5.5 velocity=50.26548246
- joint lr_tibia_pitch: limit lower=0.0 upper=2.53073 effort=5.5 velocity=50.26548246 -> lower=-0.95 upper=1.75 effort=5.5 velocity=50.26548246
- joint rf_femur_pitch: limit lower=0.0 upper=1.74533 effort=5.5 velocity=50.26548246 -> lower=-1.745329 upper=0.55 effort=5.5 velocity=50.26548246
- joint rf_tibia_pitch: limit lower=0.0 upper=2.53073 effort=5.5 velocity=50.26548246 -> lower=-0.95 upper=1.75 effort=5.5 velocity=50.26548246
- joint rm_femur_pitch: limit lower=0.0 upper=1.74533 effort=5.5 velocity=50.26548246 -> lower=-1.745329 upper=0.55 effort=5.5 velocity=50.26548246
- joint rm_tibia_pitch: limit lower=0.0 upper=2.53073 effort=5.5 velocity=50.26548246 -> lower=-0.95 upper=1.75 effort=5.5 velocity=50.26548246
- joint rr_femur_pitch: limit lower=0.0 upper=1.74533 effort=5.5 velocity=50.26548246 -> lower=-1.745329 upper=0.55 effort=5.5 velocity=50.26548246
- joint rr_tibia_pitch: limit lower=0.0 upper=2.53073 effort=5.5 velocity=50.26548246 -> lower=-0.95 upper=1.75 effort=5.5 velocity=50.26548246
