Commit message: Adopt reviewed detailed CAD as canonical training URDF

File: robot/hexapod_mkii_updated_v1/urdf/hexapod_updated_inspection.urdf (robot description, URDF)
Before this commit: robot hexapod_updated_direct_drive_inspection, 19 links, 18 joints
Joints:
- joint lf_coxa_yaw: limit lower=-0.43633231299858238 upper=0.43633231299858238 effort=0 velocity=0.5 -> lower=-1.2966923677691873 upper=1.2966923677691873 effort=0 velocity=0.5; origin xyz=0.079974503128936378 -0.199902994827965 0.028250030527750904 rpy=-0 -0 -1.1902892749824068 -> xyz=0.079974503128936378 -0.199902994827965 0.028250030527750904 rpy=0 0 -0.88514373014892411
- joint lf_femur_pitch: limit lower=-0.3490658503988659 upper=0.3490658503988659 effort=0 velocity=0.5 -> lower=-2.0943951023931953 upper=1.3962634015954636 effort=0 velocity=0.5
- joint lf_tibia_pitch: limit lower=-0.05235987755982989 upper=0.3490658503988659 effort=0 velocity=0.5 -> lower=-0.087266462599716474 upper=3.1415926535897931 effort=0 velocity=0.5
- joint lm_coxa_yaw: limit lower=-0.43633231299858238 upper=0.43633231299858238 effort=0 velocity=0.5 -> lower=-0.81533056006915106 upper=0.81533056006915106 effort=0 velocity=0.5; origin xyz=0.11997399851761598 9.7120160266750126e-05 0.028250030526969751 rpy=0 -0 6.8475982839115914e-07 -> xyz=0.11997399851761598 9.7120160266750126e-05 0.028250030526969751 rpy=0 0 -0.0089884456477707982
- joint lm_femur_pitch: limit lower=-0.3490658503988659 upper=0.3490658503988659 effort=0 velocity=0.5 -> lower=-2.0943951023931953 upper=1.3962634015954636 effort=0 velocity=0.5
- joint lm_tibia_pitch: limit lower=-0.05235987755982989 upper=0.3490658503988659 effort=0 velocity=0.5 -> lower=-0.087266462599716474 upper=3.1415926535897931 effort=0 velocity=0.5
- joint lr_coxa_yaw: limit lower=-0.43633231299858238 upper=0.43633231299858238 effort=0 velocity=0.5 -> lower=-1.3046336158657614 upper=1.3046336158657614 effort=0 velocity=0.5; origin xyz=0.079974494811767702 0.2000970031020049 0.028250019015532757 rpy=0 -0 1.1902891941000178 -> xyz=0.079974494811767702 0.2000970031020049 0.028250019015532757 rpy=0 -0 0.87510808694995645
- joint lr_femur_pitch: limit lower=-0.3490658503988659 upper=0.3490658503988659 effort=0 velocity=0.5 -> lower=-2.0943951023931953 upper=1.3962634015954636 effort=0 velocity=0.5
- joint lr_tibia_pitch: limit lower=-0.05235987755982989 upper=0.3490658503988659 effort=0 velocity=0.5 -> lower=-0.087266462599716474 upper=3.1415926535897931 effort=0 velocity=0.5
- joint rf_coxa_yaw: limit lower=-0.43633231299858238 upper=0.43633231299858238 effort=0 velocity=0.5 -> lower=-1.3046336158657614 upper=1.3046336158657614 effort=0 velocity=0.5; origin xyz=-0.080025494953448406 -0.19990300332753749 0.02825003052689477 rpy=0 -0 -1.9513018931236898 -> xyz=-0.080025494953448406 -0.19990300332753749 0.02825003052689477 rpy=0 -0 -2.2664845666398361
- joint rf_femur_pitch: limit lower=-0.3490658503988659 upper=0.3490658503988659 effort=0 velocity=0.5 -> lower=-2.0943951023931953 upper=1.3962634015954636 effort=0 velocity=0.5
- joint rf_tibia_pitch: limit lower=-0.05235987755982989 upper=0.3490658503988659 effort=0 velocity=0.5 -> lower=-0.087266462599716474 upper=3.1415926535897931 effort=0 velocity=0.5
- joint rm_coxa_yaw: limit lower=-0.43633231299858238 upper=0.43633231299858238 effort=0 velocity=0.5 -> lower=-0.81533056006915094 upper=0.81533056006915094 effort=0 velocity=0.5; origin xyz=-0.1200259984620559 9.7108454068357857e-05 0.028250030526966504 rpy=0 -0 3.141592066385154 -> xyz=-0.1200259984620559 9.7108454068357857e-05 0.028250030526966504 rpy=0 -0 3.132604207942022
- joint rm_femur_pitch: limit lower=-0.3490658503988659 upper=0.3490658503988659 effort=0 velocity=0.5 -> lower=-2.0943951023931953 upper=1.3962634015954636 effort=0 velocity=0.5
- joint rm_tibia_pitch: limit lower=-0.05235987755982989 upper=0.3490658503988659 effort=0 velocity=0.5 -> lower=-0.087266462599716474 upper=3.1415926535897931 effort=0 velocity=0.5
- joint rr_coxa_yaw: limit lower=-0.43633231299858238 upper=0.43633231299858238 effort=0 velocity=0.5 -> lower=-1.2966923677691873 upper=1.2966923677691873 effort=0 velocity=0.5; origin xyz=-0.080025502213655203 0.20009699437506273 0.02825001279546957 rpy=0 -0 1.9513020708504265 -> xyz=-0.080025502213655203 0.20009699437506273 0.02825001279546957 rpy=0 -0 2.2564489234408689
- joint rr_femur_pitch: limit lower=-0.3490658503988659 upper=0.3490658503988659 effort=0 velocity=0.5 -> lower=-2.0943951023931953 upper=1.3962634015954636 effort=0 velocity=0.5
- joint rr_tibia_pitch: limit lower=-0.05235987755982989 upper=0.3490658503988659 effort=0 velocity=0.5 -> lower=-0.087266462599716474 upper=3.1415926535897931 effort=0 velocity=0.5
